Commit message: 1

File: lprc_robot_description/urdf/mech/base.urdf.xacro (robot description, xacro)
@@ -38,9 +38,14 @@
       </visual>
     </gazebo>
-    <joint name="base_to_footprint" type="fixed">
-      <parent link="base_footprint"/>
-      <child link="base_link"/>
+    <joint name="footprint_to_base" type="fixed">
+      <parent link="base_link"/>
+      <child link="base_footprint"/>
+      <origin xyz="0 0 0" rpy="0 0 0"/>
+    </joint>
+    <!-- <joint name="base_to_footprint" type="fixed">
+      <parent link="base_link"/>
+      <child link="base_footprint"/>
       <origin xyz="0 0 ${wheel_radius - wheel_pos_z}" rpy="0 0 0"/>
-    </joint>
+    </joint> -->
   </xacro:macro>
 </robot>

File: lprc_robot_description/urdf/robots/mecanum.urdf.xacro (robot description, xacro)
@@ -6,5 +6,4 @@
   <xacro:include filename="$(find linorobot2_description)/urdf/sensors/imu.urdf.xacro" />
   <xacro:include filename="$(find linorobot2_description)/urdf/sensors/generic_laser.urdf.xacro" />
-  <xacro:include filename="$(find linorobot2_description)/urdf/sensors/depth_sensor.urdf.xacro" />
   <xacro:include filename="$(find linorobot2_description)/urdf/controllers/omni_drive.urdf.xacro" />
   <xacro:base
@@ -56,7 +55,4 @@
     <xacro:insert_block name="laser_pose" />
   </xacro:generic_laser>
-  <xacro:depth_sensor>
-    <xacro:insert_block name="depth_sensor_pose" />
-  </xacro:depth_sensor>
   <xacro:omni_drive_controller/>
 </robot>
